File: kicad/kint.kicad_pcb (KiCad board)
At the start: 2 copper layers, 107.9 x 86 mm, 27 parts, among them J1 THUMB_RIGHT_SPC_KB600, J2 LEFT_13_LT, J3 TOP_LEFT, J4 TOP_RIGHT, J5 THUMB_LEFT_BAK, J6 THUMB_RIGHT_SPC, J7 RIGHT_13_DOWN, J8 THUMB_LEFT_BAK_KB600, U1 TEENSY_3.5_3.6

Commit message: Fix up board and schematic in KiCad
Not too bad, I think the merging was worth it
Connections:
- J1 pad 1: Net-(J1-Pad1) -> unconnected-(J1-Pad1)
- J1 pad 10: Net-(J1-Pad10) -> unconnected-(J1-Pad10)
- J1 pad 11: Net-(J1-Pad11) -> unconnected-(J1-Pad11)
- J1 pad 12: Net-(J1-Pad12) -> unconnected-(J1-Pad12)
- J1 pad 13: Net-(J1-Pad13) -> unconnected-(J1-Pad13)
- J1 pad 2: Net-(J1-Pad2) -> unconnected-(J1-Pad2)
- J1 pad 9: Net-(J1-Pad9) -> unconnected-(J1-Pad9)
- J2 pad 10: Net-(J2-Pad10) -> unconnected-(J2-Pad10)
- J2 pad 5: Net-(J2-Pad5) -> unconnected-(J2-Pad5)
- J3 pad 12: Net-(J3-Pad12) -> unconnected-(J3-Pad12)
- J3 pad 13: Net-(J3-Pad13) -> unconnected-(J3-Pad13)
- J3 pad 9: Net-(J3-Pad9) -> unconnected-(J3-Pad9)
- J4 pad 1: Net-(J4-Pad1) -> unconnected-(J4-Pad1)
- J4 pad 2: Net-(J4-Pad2) -> unconnected-(J4-Pad2)
- J5 pad 10: Net-(J5-Pad10) -> unconnected-(J5-Pad10)
- J5 pad 6: Net-(J5-Pad6) -> unconnected-(J5-Pad6)
- J5 pad 7: Net-(J5-Pad7) -> unconnected-(J5-Pad7)
- J5 pad 9: Net-(J5-Pad9) -> unconnected-(J5-Pad9)
- J6 pad 1: Net-(J6-Pad1) -> unconnected-(J6-Pad1)
- J6 pad 10: Net-(J6-Pad10) -> unconnected-(J6-Pad10)
- J6 pad 2: Net-(J6-Pad2) -> unconnected-(J6-Pad2)
- J6 pad 9: Net-(J6-Pad9) -> unconnected-(J6-Pad9)
- J7 pad 11: Net-(J7-Pad11) -> unconnected-(J7-Pad11)
- J7 pad 5: Net-(J7-Pad5) -> unconnected-(J7-Pad5)
- J8 pad 1: Net-(J8-Pad1) -> unconnected-(J8-Pad1)
- J8 pad 2: Net-(J8-Pad2) -> unconnected-(J8-Pad2)
- J8 pad 3: Net-(J8-Pad3) -> unconnected-(J8-Pad3)
- J8 pad 4: Net-(J8-Pad4) -> unconnected-(J8-Pad4)
- J8 pad 5: Net-(J8-Pad5) -> unconnected-(J8-Pad5)
- J8 pad 7: Net-(J8-Pad7) -> unconnected-(J8-Pad7)
- J8 pad 8: Net-(J8-Pad8) -> unconnected-(J8-Pad8)
- JP1 pad 1: (no net) -> Net-(JP1-Pad1)
- JP5 pad 1: Net-(JP2-Pad1) -> Net-(JP5-Pad1)
- JP5 pad 2: /ROW_4 -> /ROW_5
- U1 pad 13/SCK: Net-(U1-Pad13/SCK) -> unconnected-(U1-Pad13/SCK)
- U1 pad 21/DAC0: Net-(U1-Pad21/DAC0) -> unconnected-(U1-Pad21/DAC0)
- U1 pad 28: Net-(U1-Pad28) -> unconnected-(U1-Pad28)
- U1 pad 29: Net-(U1-Pad29) -> unconnected-(U1-Pad29)
- U1 pad 30: Net-(U1-Pad30) -> unconnected-(U1-Pad30)
- U1 pad 31/A12: Net-(U1-Pad31/A12) -> unconnected-(U1-Pad31/A12)
- U1 pad 32/A13: Net-(U1-Pad32/A13) -> unconnected-(U1-Pad32/A13)
- U1 pad 33/A14: Net-(U1-Pad33/A14) -> unconnected-(U1-Pad33/A14)
- U1 pad 34/A15: Net-(U1-Pad34/A15) -> unconnected-(U1-Pad34/A15)
- U1 pad 35/A16: Net-(U1-Pad35/A16) -> unconnected-(U1-Pad35/A16)
- U1 pad 36/A17: Net-(U1-Pad36/A17) -> unconnected-(U1-Pad36/A17)
- U1 pad 39/A20: Net-(U1-Pad39/A20) -> unconnected-(U1-Pad39/A20)
- U1 pad 3V3: Net-(U1-Pad3V3) -> unconnected-(U1-Pad3V3)
- U1 pad 3V3_LO: Net-(U1-Pad3V3_LO) -> unconnected-(U1-Pad3V3_LO)
- U1 pad A22/DAC1: Net-(U1-PadA22/DAC1) -> unconnected-(U1-PadA22/DAC1)
- U1 pad AGND: Net-(U1-PadAGND) -> unconnected-(U1-PadAGND)
- U1 pad GND2: Net-(U1-PadGND2) -> unconnected-(U1-PadGND2)
- U1 pad PROG: Net-(U1-PadPROG) -> unconnected-(U1-PadPROG)
- U1 pad RESET: Net-(U1-PadRESET) -> unconnected-(U1-PadRESET)
- U1 pad VBAT: Net-(U1-PadVBAT) -> unconnected-(U1-PadVBAT)
- U1 pad VIN: Net-(U1-PadVIN) -> unconnected-(U1-PadVIN)
Routing:
- net unconnected-(U1-PadRESET): track 0.00 -> 16.3 mm
- net Net-(U1-PadRESET): track 16.3 -> 0.00 mm
- net unconnected-(U1-PadVBAT): track 0.00 -> 12.7 mm
- net unconnected-(U1-PadPROG): track 0.00 -> 12.7 mm
- net Net-(U1-PadVBAT): track 12.7 -> 0.00 mm
- net Net-(U1-PadPROG): track 12.7 -> 0.00 mm
- net (no net): track 8.59 -> 0.00 mm
